File: hardware/RSMS_Kicad/RSMS_Kicad.kicad_pcb (KiCad board)
At the start: 2 copper layers, 35 x 30 mm, 16 parts, among them J2 INTF1, J3 INTF2, U1 ESP32-S2-WROOM, U3 AMS1117-3.3

Commit message: update repo
Parts:
- U1: value ESP32-S2-WROOM -> ESP32-WROOM-32; footprint ESP32-S2-WROOM:ESP32-S2-WROOM -> RF_Module:ESP32-WROOM-32
- U3: moved to F.Cu
- moved C2 40.7 mm to (122.9, 121.6)
- moved R7 40.7 mm to (122.9, 119.6)
- moved S2 40.7 mm to (127.5, 120.8)
- moved D1 25.5 mm to (131.6, 82.3), turned to 0 degrees
- moved R5 23.2 mm to (131.4, 84.1), turned to 180 degrees
- moved C1 21.0 mm to (146.4, 82.2), turned to 90 degrees
- moved U3 19.4 mm to (125.2, 85.5), turned to 0 degrees
- moved R6 19.0 mm to (144.3, 82.2), turned to -90 degrees
- moved C3 17.0 mm to (126.2, 91.2), turned to -90 degrees
- moved C4 14.4 mm to (128.4, 91.6), turned to -90 degrees
- moved S1 10.5 mm to (140.5, 82.3), turned to 0 degrees
- moved U1 8.62 mm to (141.4, 95.0), turned to -90 degrees
- moved D2 8.18 mm to (136.4, 107.1)
- moved R8 8.18 mm to (134.6, 106.8)
Connections:
- U1 pad 15: unconnected-(U1-Pad15) -> GND
- U1 pad 26: GND -> unconnected-(U1-Pad26)
- U1 pad 27: unconnected-(U1-Pad27) -> /R_TX
- U1 pad 28: unconnected-(U1-Pad28) -> /R_RX
- U1 pad 3: unconnected-(U1-Pad3) -> /nRST
- U1 pad 38: unconnected-(U1-Pad38) -> GND
- U1 pad 39: unconnected-(U1-Pad39) -> GND
Routing:
- net /R_TX: track 0.00 -> 23.6 mm, vias 0 -> 1
- net /R_RX: track 0.00 -> 20.9 mm, vias 0 -> 1
- net +3V3: track 21.7 -> 11.3 mm, vias 2 -> 0
- net VBUS: track 0.00 -> 7.82 mm, vias 0 -> 3
- net /nRST: track 6.48 -> 7.90 mm
- added copper zone on F.Cu, net +3V3
- added copper zone on B.Cu, net VBUS
