File: hardware/RSMS_Kicad/RSMS_Kicad.kicad_sch (KiCad schematic)
At the start: 16 parts, among them J2 INTF1, J3 INTF2, U1 ESP32-S2-WROOM, U3 AMS1117-3.3

Commit message: update repo
Parts:
- removed U1: ESP32-S2-WROOM, ESP32-S2-WROOM:ESP32-S2-WROOM, symbol ESP32-S2-WROOM:ESP32-S2-WROOM
- added U1: ESP32-WROOM-32, RF_Module:ESP32-WROOM-32, symbol RF_Module:ESP32-WROOM-32
Connections:
- net +3V3: now also U1.2 (VDD)
- net GND: now also U1.1 (GND), U1.15 (GND), U1.38 (GND), U1.39 (GND)
- net R_RX: now also U1.28 (IO17)
- net R_TX: now also U1.27 (IO16)
- net nRST: now also U1.3 (EN)
